File: pcb/uart384.kicad_sch (KiCad schematic)
At the start: 32 parts, among them IC1 ICE40LP384-SG32, J1 USB_A, J2 TC2050, J3 Conn_02x06_Odd_Even, SW1 SW_Push, U1 CP2102-QFN28, U2 AT25DF256-XMHN-T, U3 MIC5365-1.2YC5, Y1 XO32

Commit message: release PCB v1.0: setup production files, docs
Other:
- title: (none) -> UART384
Changed lines of the file:
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@@
 	(generator_version "9.0")
 	(paper "A4")
+	(title_block
+		(title "UART384")
+		(date "2025-08-26")
+		(rev "v1.0")
+		(comment 1 "a USB/UART enabled dev-board for the ice40LP384")
+		(comment 2 "https://github.com/dpiegdon/uart384")
+	)
 	(text "Close to VCCIO pins"
 		(exclude_from_sim no)
